Commit message: Add T800 RL recovery training pipeline

File: GMR/assets/t800/serial_t800.urdf (robot description, URDF)
Before this commit: robot t800, 30 links, 29 joints
Links:
- link LINK_ANKLE_PITCH_L: geometry visual mesh filename=meshes/LINK_ANKLE_PITCH_L.dae
- link LINK_ANKLE_PITCH_R: geometry visual mesh filename=meshes/LINK_ANKLE_PITCH_R.dae
- link LINK_ANKLE_ROLL_L: geometry collision box size=0.26 0.10 0.02; visual mesh filename=meshes/LINK_ANKLE_ROLL_L.dae
- link LINK_ANKLE_ROLL_R: geometry collision box size=0.26 0.10 0.02; visual mesh filename=meshes/LINK_ANKLE_ROLL_R.dae
- link LINK_BASE: geometry collision sphere radius=0.09; visual mesh filename=meshes/LINK_BASE.dae
- link LINK_ELBOW_PITCH_L: geometry collision sphere radius=0.05; visual mesh filename=meshes/LINK_ELBOW_PITCH_L.dae
- link LINK_ELBOW_PITCH_R: geometry collision sphere radius=0.05; visual mesh filename=meshes/LINK_ELBOW_PITCH_R.dae
- link LINK_ELBOW_YAW_L: geometry collision box size=0.08 0.08 0.14; visual mesh filename=meshes/LINK_ELBOW_YAW_L.dae
- link LINK_ELBOW_YAW_R: geometry collision box size=0.08 0.08 0.14; visual mesh filename=meshes/LINK_ELBOW_YAW_R.dae
- link LINK_HEAD_PITCH: geometry visual mesh filename=meshes/LINK_HEAD_PITCH.dae
- link LINK_HEAD_YAW: geometry collision sphere radius=0.08; visual mesh filename=meshes/LINK_HEAD_YAW.dae
- link LINK_HIP_PITCH_L: geometry collision sphere radius=0.07; visual mesh filename=meshes/LINK_HIP_PITCH_L.dae
- link LINK_HIP_PITCH_R: geometry collision sphere radius=0.07; visual mesh filename=meshes/LINK_HIP_PITCH_R.dae
- link LINK_HIP_ROLL_L: geometry visual mesh filename=meshes/LINK_HIP_ROLL_L.dae
- link LINK_HIP_ROLL_R: geometry visual mesh filename=meshes/LINK_HIP_ROLL_R.dae
- link LINK_HIP_YAW_L: geometry collision box size=0.10 0.12 0.18; visual mesh filename=meshes/LINK_HIP_YAW_L.dae
- link LINK_HIP_YAW_R: geometry collision box size=0.10 0.12 0.18; visual mesh filename=meshes/LINK_HIP_YAW_R.dae
- link LINK_KNEE_PITCH_L: geometry collision box size=0.11 0.09 0.24; collision sphere radius=0.08
- link LINK_KNEE_PITCH_R: geometry collision box size=0.11 0.09 0.23; collision sphere radius=0.08
- link LINK_SHOULDER_PITCH_L: geometry collision sphere radius=0.06; visual mesh filename=meshes/LINK_SHOULDER_PITCH_L.dae
- link LINK_SHOULDER_PITCH_R: geometry collision sphere radius=0.06; visual mesh filename=meshes/LINK_SHOULDER_PITCH_R.dae
- link LINK_SHOULDER_ROLL_L: geometry visual mesh filename=meshes/LINK_SHOULDER_ROLL_L.dae
- link LINK_SHOULDER_ROLL_R: geometry visual mesh filename=meshes/LINK_SHOULDER_ROLL_R.dae
- link LINK_SHOULDER_YAW_L: geometry collision box size=0.08 0.08 0.10; visual mesh filename=meshes/LINK_SHOULDER_YAW_L.dae
- link LINK_SHOULDER_YAW_R: geometry collision box size=0.08 0.08 0.10; visual mesh filename=meshes/LINK_SHOULDER_YAW_R.dae
- link LINK_TORSO_YAW: geometry collision box size=0.18 0.20 0.14; collision box size=0.22 0.28 0.19
